File: Schaltplan/Schaltplan.kicad_sch (KiCad schematic)
At the start: 2 parts, among them U1 LTC6804-1, U2 TLP175A

Commit message: Commit
Parts:
- removed U1: LTC6804-1, Package_SO:SSOP-48_5.3x12.8mm_P0.5mm, symbol Battery_Management:LTC6804-1
- removed U2: TLP175A, Package_SO:Toshiba_SOIC-4-6_4.4x3.6mm_P1.27mm, symbol Relay_SolidState:TLP175A
- added A1: Arduino_Nano, Module:Arduino_Nano, symbol MCU_Module:Arduino_Nano_v3.x
- added BT1, BT2: Battery_Cell, symbol Device:Battery_Cell
- added J1: Conn_01x02_Pin, symbol Connector:Conn_01x02_Pin
- added Q1, Q2: IRLZ44N, Package_TO_SOT_THT:TO-220-3_Vertical, symbol Transistor_FET:IRLZ44N
- added R1, R2, R3, R4, R5, R6, R7: R, symbol Device:R
Connections:
- new net: BT1.1 (+), BT2.2 (-), R1.1
- new net: A1.19 (A0), R1.2, R2.2
- new net: A1.2 (D0/RX), A1.4 (GND), BT1.2 (-), Q1.2 (D), Q2.2 (D), R2.1, R6.2, R7.2
- new net: Q1.1 (G), R3.1
- new net: A1.8 (D5), R3.2, R6.1
- new net: A1.30 (VIN), BT2.1 (+), J1.1 (Pin_1), R5.1
- new net: J1.2 (Pin_2), Q1.3 (S), Q2.3 (S)
- new net: Q2.1 (G), R4.1
- new net: A1.9 (D6), R4.2, R7.1
- new net: A1.20 (A1), R5.2
Other:
- company: (none) -> AkkuCraft
- title: (none) -> Schaltplan Powerbank
